File: SCHEMATIC/schematic.kicad_sch (KiCad schematic)
At the start: 83 parts, among them J1 12V_AC_IN, K1 Relay_SPST-NO, K2 Relay_SPST-NO, K3 Relay_SPST-NO, Q1 2N2219/INVERTER, Q2 2N2219, Q3 2N2219, U1 L7805, U10 74HC74, U11 SN74HC163N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

Commit message: Add files via upload
Fixed errors in schematic
Parts:
- removed unit 2 of F1
- renumbered U3 to F1, U5 to F2, U6 to U5
Connections:
- net 50HZ_CLK: now also F1.7; no longer F1.1
- net GND: now also F1.6 (-); no longer F1.2 (-)
- net at D2.1 (K), R3.2: now also F1.5 (+); no longer F1.3 (+)
- net ST00: no longer names the net of U8.3 (1Y)
- net ST01: no longer names the net of U8.6 (2Y)
- net ST10: no longer names the net of U8.8 (3Y)
- net ST11: no longer names the net of U8.11 (4Y)
- no-connect marks 0 -> 37
Other:
- note added: "Reference High"
- note added: "Reference Low"
